File: hardware/KiCad/nonisolated.kicad_sch (KiCad schematic)
At the start: 2 parts, among them P401 BNC

Commit message: Version 2.0
1wire sensor
flow sensor
Parts:
- removed P401: BNC, temp_terminal:WL-EB08040502_snk, symbol tentacle-raspi:BNC
- removed STP401: EZO_SMD, temp_terminal:WL-ezo-smd, symbol tentacle-raspi:EZO_SMD
- added J1, J2: Conn_01x03, Connector_Phoenix_MC:PhoenixContact_MC_1,5_3-G-3.5_1x03_P3.50mm_Horizontal, symbol Connector_Generic:Conn_01x03
- added R1, R2: 4.7K, temp_terminal:WL-SM0805R, symbol tentacle-raspi:R
Connections:
- net +3.3V: now also J1.3 (Pin_3), J2.3 (Pin_3), R1.2, R2.2
- net GND: now also J1.1 (Pin_1), J2.1 (Pin_1)
- new net FLOW: J2.2 (Pin_2), R1.1
- new net TEMP: J1.2 (Pin_2), R2.1
Other:
- note removed: "NC"
- note removed: "PT-1000"
- note removed: "probe +"
- note removed: "probe -"
