File: hardware/KiCad/tentacle-raspi.kicad_sch (KiCad schematic)
At the start: 6 parts, among them P101 CONN_01X06, P102 CONN_01X06

Commit message: Version 2.0
1wire sensor
flow sensor
Parts:
- removed P102: CONN_01X06, temp_terminal:WL-PINH_1X6_snk, symbol tentacle-raspi:CONN_01X06
Connections:
- net nonisolated1/TEMP: now reaches PI_BOARD101.33 (GPIO13)
- net nonisolated1/FLOW: now reaches PI_BOARD101.37 (GPIO26)
- no-connect marks 34 -> 32
Other:
- sheet nonisolated1 ports: added FLOW, TEMP; removed RX, TX
- note removed: "Channel 5"
